File: hardware/_autosave-nfc_sense.kicad_pcb (KiCad board)
At the start: 2 copper layers, 18.6 x 35.8 mm, 22 parts, among them U1 TMP112AIDRLT, U2 RF430CL330HIRGTR‎, U3 ATtiny3227-M

Commit message: triangle extension
Parts:
- renumbered GND to GND1, UPDI to UPDI1, VCC to VCC1
Other:
- board size 18.6 x 35.8 mm -> 18.6 x 44.5 mm
Changed lines of the file:
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@@
     (property "Sheetname" "")
     (attr through_hole)
-    (fp_text reference "AE1" (at 0.9 -1.9 unlocked) (layer "F.SilkS")
-      (effects (font (size 0.75 0.75) (thickness 0.125)))
-    )
-    (fp_text value "Antenna_Dipole" (at 8.3 -1.8 unlocked) (layer "F.Fab")
-      (effects (font (size 1 1) (thickness 0.15)))
-    )
-    (fp_line (start -1 -1) (end 3.75 -1) (layer "B.SilkS") (width 0.1))
-    (fp_line (start 19 -1) (end 14.25 -1) (layer "B.SilkS") (width 0.1))
-    (fp_line (start 19 36) (end 19 31.25) (layer "B.SilkS") (width 0.1))
-    (fp_line (start -1 36) (end 3.75 36) (layer "B.SilkS") (width 0.1))
-    (fp_line (start -1 -1) (end -1 3.75) (layer "B.SilkS") (width 0.1))
-    (fp_line (start 19 -1) (end 19 3.75) (layer "B.SilkS") (width 0.1))
-    (fp_line (start 19 36) (end 14.25 36) (layer "B.SilkS") (width 0.1))
-    (fp_line (start -1 36) (end -1 31.25) (layer "B.SilkS") (width 0.1))
-    (fp_line (start -1 -1) (end 19 -1) (layer "F.SilkS") (width 0.1))
-    (fp_line (start 19 36) (end -1 36) (layer "F.SilkS") (width 0.1))
-    (fp_line (start -1 36) (end -1 -1) (layer "F.SilkS") (width 0.1))
-    (fp_line (start 19 -1) (end 19 36) (layer "F.SilkS") (width 0.1))
-    (pad "1" thru_hole circle (at 8.12868 34.875) (size 0.5 0.5) (drill 0.25) (layers *.Cu *.Mask)
-      (net 3 "ANT1") (pintype "input"))
+    (fp_text reference "AE1" (at 0.9 -1.9) (layer "F.SilkS")
+      (effects (font (size 0.75 0.75) (thickness 0.125)))
+    )
+    (fp_text value "Antenna_Dipole" (at 8.3 -1.8) (layer "F.Fab")
+      (effects (font (size 1 1) (thickness 0.15)))
+    )
     (pad "1" smd custom (at 8.12868 34.875) (size 0.25 0.25) (layers "F.Cu")
       (net 3 "ANT1") (pintype "input") (zone_connect 0)
@@
         (gr_line (start 7.24632 -32.25) (end 7.24632 -2.5) (width 0.25))
       ))
-    (pad "2" thru_hole circle (at 9.87132 32.375) (size 0.5 0.5) (drill 0.25) (layers *.Cu *.Mask)
-      (net 2 "ANT2") (pintype "input"))
+    (pad "1" thru_hole circle (at 8.12868 34.875) (size 0.5 0.5) (drill 0.25) (layers *.Cu *.Mask)
+      (net 3 "ANT1") (pintype "input"))
     (pad "2" smd custom (at 9.87132 32.375) (size 0.25 0.25) (layers "F.Cu")
       (net 2 "ANT2") (pintype "input") (zone_connect 0)
@@
         (gr_line (start 0 0) (end 5.50368 0) (width 0.25))
       ))
+    (pad "2" thru_hole circle (at 9.87132 32.375) (size 0.5 0.5) (drill 0.25) (layers *.Cu *.Mask)
+      (net 2 "ANT2") (pintype "input"))
   )
   (footprint "unsurv_offline_pcb_footprints:RF430_3x3mm_noBCu" (layer "F.Cu")
@@
     (property "Sheetname" "")
     (attr exclude_from_pos_files)
-    (fp_text reference "VCC" (at -0.1 -2.5 unlocked) (layer "B.SilkS")
+    (fp_text reference "VCC1" (at -0.1 -2.5 unlocked) (layer "B.SilkS")
       (effects (font (size 0.75 0.75) (thickness 0.125)) (justify mirror))
     )
@@
     (property "Sheetname" "")
     (attr exclude_from_pos_files)
-    (fp_text reference "UPDI" (at 0 -2.6 unlocked) (layer "B.SilkS")
+    (fp_text reference "UPDI1" (at 0 -2.6 unlocked) (layer "B.SilkS")
       (effects (font (size 0.75 0.75) (thickness 0.125)) (justify mirror))
     )
@@
     (property "Sheetname" "")
     (attr exclude_from_pos_files)
-    (fp_text reference "GND" (at 0 -2.5 unlocked) (layer "B.SilkS")
+    (fp_text reference "GND1" (at 0 -2.5 unlocked) (layer "B.SilkS")
       (effects (font (size 0.75 0.75) (thickness 0.125)) (justify mirror))
     )
@@
   )
   (gr_circle (center 123.95 47) (end 123.9 47.1) (layer "F.SilkS") (width 0.1) (fill none))
-  (gr_line (start 138.299999 67.25) (end 120.699999 67.25) (layer "Edge.Cuts") (width 0.1))
+  (gr_arc (start 129.95 75.8) (mid 129.5 75.986396) (end 129.05 75.8) (layer "Edge.Cuts") (width 0.1))
   (gr_arc (start 128.8 41.099999) (mid 129.5 37.175155) (end 130.2 41.099999) (layer "Edge.Cuts") (width 0.1))
   (gr_arc (start 128.8 42.999999) (mid 129.5 35.336033) (end 130.2 42.999999) (layer "Edge.Cuts") (width 0.1))
   (gr_line (start 120.699999 31.499999) (end 138.299999 31.499999) (layer "Edge.Cuts") (width 0.1))
+  (gr_circle (center 129.5 71.15) (end 131.5 71.15) (layer "Edge.Cuts") (width 0.1) (fill none))
   (gr_arc (start 120.199999 31.999999) (mid 120.346446 31.646446) (end 120.699999 31.499999) (layer "Edge.Cuts") (width 0.1))
   (gr_line (start 128.8 42.999999) (end 128.8 41.099998) (layer "Edge.Cuts") (width 0.1))
-  (gr_arc (start 120.699999 67.246447) (mid 120.34643 67.100003) (end 120.199999 66.746447) (layer "Edge.Cuts") (width 0.1))
+  (gr_arc (start 120.34643 67.100003) (mid 120.238047 66.93779) (end 120.199999 66.746447) (layer "Edge.Cuts") (width 0.1))
   (gr_line (start 138.799999 31.999999) (end 138.799999 66.746447) (layer "Edge.Cuts") (width 0.1))
   (gr_arc (start 138.299999 31.499999) (mid 138.653553 31.646445) (end 138.799999 31.999999) (layer "Edge.Cuts") (width 0.1))
   (gr_line (start 120.199999 66.746447) (end 120.199999 31.999999) (layer "Edge.Cuts") (width 0.1))
   (gr_line (start 130.2 41.099999) (end 130.2 42.999999) (layer "Edge.Cuts") (width 0.1))
-  (gr_arc (start 138.799999 66.746447) (mid 138.653536 67.09997) (end 138.299999 67.246447) (layer "Edge.Cuts") (width 0.1))
+  (gr_line (start 138.653536 67.09997) (end 129.95 75.8) (layer "Edge.Cuts") (width 0.1))
+  (gr_arc (start 138.799999 66.746447) (mid 138.761923 66.937773) (end 138.653536 67.09997) (layer "Edge.Cuts") (width 0.1))
+  (gr_line (start 129.05 75.8) (end 120.34643 67.100003) (layer "Edge.Cuts") (width 0.1))
   (segment (start 133.98821 54.91179) (end 133.25 54.91179) (width 0.2) (layer "F.Cu") (net 1))
   (segment (start 129.5 39.3) (end 129.5 38.9) (width 0.2) (layer "F.Cu") (net 1))
