File: hardware/nfc_sense.kicad_sch (KiCad schematic)
At the start: 25 parts, among them U1 TMP117AIDRVR, U2 RF430CL330HIRGTR‎, U3 ATtiny1626-MFR

Commit message: change footprints for better paste application
Parts:
- D1, D2: footprint Diode_SMD:D_0603_1608Metric_Pad1.05x0.95mm_HandSolder -> Diode_SMD:D_0603_1608Metric
- R1, R2: footprint Resistor_SMD:R_0603_1608Metric_Pad0.98x0.95mm_HandSolder -> Resistor_SMD:R_0603_1608Metric
- U2: footprint unsurv_offline_pcb_footprints:RF430_3x3mm_noBCu -> unsurv_offline_pcb_footprints:RF430_3x3mm_regular
- U3: footprint Package_DFN_QFN:VQFN-20-1EP_3x3mm_P0.4mm_EP1.7x1.7mm -> unsurv_offline_pcb_footprints:VQFN-20-1EP_3x3mm_P0.4mm_EP1.7x1.7mm_edited
Changed lines of the file:
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@@
 			)
 		)
-		(property "Footprint" "unsurv_offline_pcb_footprints:RF430_3x3mm_noBCu"
+		(property "Footprint" "unsurv_offline_pcb_footprints:RF430_3x3mm_regular"
 			(at 59.69 26.035 0)
 			(effects
@@
 			)
 		)
-		(property "Footprint" "Diode_SMD:D_0603_1608Metric_Pad1.05x0.95mm_HandSolder"
+		(property "Footprint" "Diode_SMD:D_0603_1608Metric"
 			(at 113.665 60.96 0)
 			(effects
@@
 			)
 		)
-		(property "Footprint" "Diode_SMD:D_0603_1608Metric_Pad1.05x0.95mm_HandSolder"
+		(property "Footprint" "Diode_SMD:D_0603_1608Metric"
 			(at 114.3 46.355 0)
 			(effects
@@
 			)
 		)
-		(property "Footprint" "Resistor_SMD:R_0603_1608Metric_Pad0.98x0.95mm_HandSolder"
+		(property "Footprint" "Resistor_SMD:R_0603_1608Metric"
 			(at 147.447 87.63 90)
 			(effects
@@
 			)
 		)
-		(property "Footprint" "Resistor_SMD:R_0603_1608Metric_Pad0.98x0.95mm_HandSolder"
+		(property "Footprint" "Resistor_SMD:R_0603_1608Metric"
 			(at 137.287 87.63 90)
 			(effects
@@
 			)
 		)
-		(property "Footprint" "Package_DFN_QFN:VQFN-20-1EP_3x3mm_P0.4mm_EP1.7x1.7mm"
+		(property "Footprint" "unsurv_offline_pcb_footprints:VQFN-20-1EP_3x3mm_P0.4mm_EP1.7x1.7mm_edited"
 			(at 64.77 131.445 0)
 			(effects

Commit message: update RF430 footprint
Parts:
- U2: footprint unsurv_offline_pcb_footprints:RF430_3x3mm_regular -> unsurv_offline_pcb_footprints:RF430_3x3mm_regular_noBCu
Changed lines of the file:
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@@
 			)
 		)
-		(property "Footprint" "unsurv_offline_pcb_footprints:RF430_3x3mm_regular"
+		(property "Footprint" "unsurv_offline_pcb_footprints:RF430_3x3mm_regular_noBCu"
 			(at 59.69 26.035 0)
 			(effects
