File: hardware/nfc_victorinox/victorinox_sense.kicad_sch (KiCad schematic)
At the start: 24 parts, among them U1 TMP117AIDRVR, U2 RF430CL330HIRGTR‎, U3 ATtiny1626-MFR

Commit message: flip antenna layer, fix ANT connection issues
Connections:
- net ANT1: now also AE1.1; no longer AE1.2
- net ANT2: now also AE1.2; no longer AE1.1
Changed lines of the file:
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@@
 	(global_label "ANT2"
 		(shape input)
-		(at 170.18 48.26 0)
+		(at 162.56 48.26 180)
 		(fields_autoplaced yes)
 		(effects
@@
 				(size 1.27 1.27)
 			)
-			(justify left)
+			(justify right)
 		)
 		(property "Intersheetrefs" "${INTERSHEET_REFS}"
-			(at 177.7614 48.26 0)
+			(at 154.9786 48.26 0)
 			(effects
 				(font
 					(size 1.27 1.27)
 				)
-				(justify left)
+				(justify right)
 				(hide yes)
 			)
@@
 	(global_label "ANT1"
 		(shape input)
-		(at 162.56 48.26 180)
+		(at 170.18 48.26 0)
 		(fields_autoplaced yes)
 		(effects
@@
 				(size 1.27 1.27)
 			)
-			(justify right)
+			(justify left)
 		)
 		(property "Intersheetrefs" "${INTERSHEET_REFS}"
-			(at 154.9786 48.26 0)
+			(at 177.7614 48.26 0)
 			(effects
 				(font
 					(size 1.27 1.27)
 				)
-				(justify right)
+				(justify left)
 				(hide yes)
 			)
