File: hardware/nfc_sense_ntag_BME/nfc_sense_ntag_BME.kicad_pcb (KiCad board)
At the start: 4 copper layers, 18.6 x 34.4 mm, 17 parts, among them U4 BME280

Commit message: finalize iOS version
Routing:
- net GND: track 43.1 -> 44.8 mm, vias 5 -> 6
- net SCL: track 16.3 -> 17.3 mm
Changed lines of the file:
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@@
 		(at 129.325001 39.025 180)
 		(property "Reference" "U4"
-			(at 0 -2.3 360)
+			(at 0 -2.3 0)
 			(layer "F.SilkS")
 			(hide yes)
@@
 		)
 		(property "Value" "BME280"
-			(at 0 2.47 360)
+			(at 0 2.47 0)
 			(layer "F.Fab")
 			(effects
@@
 		)
 		(property "Footprint" "digikey-footprints:Pressure_Sensor_LGA-8_2.5x2.5mm_BME280"
-			(at 0 0 360)
+			(at 0 0 0)
 			(layer "F.Fab")
 			(hide yes)
@@
 		)
 		(property "Datasheet" "https://ae-bst.resource.bosch.com/media/_tech/media/datasheets/BST-BME280-DS002.pdf"
-			(at 0 0 360)
+			(at 0 0 0)
 			(layer "F.Fab")
 			(hide yes)
@@
 		)
 		(property "Description" "SENSOR PRESSURE HUMIDITY TEMP"
-			(at 0 0 360)
+			(at 0 0 0)
 			(layer "F.Fab")
 			(hide yes)
@@
 		)
 		(fp_text user "${REFERENCE}"
-			(at 0 0 360)
+			(at 0 0 0)
 			(layer "F.Fab")
 			(effects
@@
 		(tags "capacitor")
 		(property "Reference" "C8"
-			(at 0 -1.16 360)
+			(at 0 -1.16 0)
 			(layer "F.SilkS")
 			(hide yes)
@@
 		)
 		(property "Value" "0.1 uF"
-			(at 0 1.16 360)
+			(at 0 1.16 0)
 			(layer "F.Fab")
 			(effects
@@
 		)
 		(fp_text user "${REFERENCE}"
-			(at 0 0 360)
+			(at 0 0 0)
 			(layer "F.Fab")
 			(effects
@@
 	)
 	(segment
+		(start 130.300001 39.5)
+		(end 130.300001 40.05)
+		(width 0.2)
+		(layer "F.Cu")
+		(net 1)
+	)
+	(segment
 		(start 129.02 41.05)
 		(end 129.02 41.03)
@@
 	)
 	(segment
-		(start 130.300001 39.400001)
-		(end 130.3 39.4)
+		(start 126 48.7)
+		(end 127.65 50.35)
 		(width 0.2)
 		(layer "F.Cu")
@@
 	)
 	(segment
-		(start 130.300001 40.05)
-		(end 130.300001 39.400001)
+		(start 128.350001 37.799999)
+		(end 128.350001 38.000001)
 		(width 0.2)
 		(layer "F.Cu")
@@
 	)
 	(segment
-		(start 126 48.7)
-		(end 127.65 50.35)
+		(start 127.65 50.35)
+		(end 128.15 50.35)
 		(width 0.2)
 		(layer "F.Cu")
@@
 	)
 	(segment
-		(start 128.350001 37.799999)
-		(end 128.350001 38.000001)
+		(start 128.55 41)
+		(end 128.35 40.8)
 		(width 0.2)
 		(layer "F.Cu")
@@
 	)
 	(segment
-		(start 127.65 50.35)
-		(end 128.15 50.35)
+		(start 129.07 41)
+		(end 129.07 40.98)
 		(width 0.2)
 		(layer "F.Cu")
@@
 	(segment
 		(start 129.07 41)
-		(end 129.07 40.98)
+		(end 128.55 41)
 		(width 0.2)
 		(layer "F.Cu")
@@
 	)
 	(via
-		(at 130.3 39.4)
+		(at 130.300001 39.5)
+		(size 0.45)
+		(drill 0.25)
+		(layers "F.Cu" "B.Cu")
+		(net 1)
+	)
+	(via
+		(at 128.35 40.8)
 		(size 0.45)
 		(drill 0.25)
@@
 	)
 	(segment
-		(start 124.7 49.1)
-		(end 124.7 48.4)
+		(start 128.55 41)
+		(end 128.35 40.8)
 		(width 0.2)
 		(layer "B.Cu")
@@
 	)
 	(segment
-		(start 130.95 38.75)
-		(end 130.95 37.95)
+		(start 129.2 41)
+		(end 128.55 41)
+		(width 0.2)
+		(layer "B.Cu")
+		(net 1)
+	)
+	(segment
+		(start 124.7 49.1)
+		(end 124.7 48.4)
 		(width 0.2)
 		(layer "B.Cu")
@@
 	)
 	(segment
+		(start 129.2 46.65)
+		(end 129.2 41)
+		(width 0.2)
+		(layer "B.Cu")
+		(net 1)
+	)
+	(segment
 		(start 132.95 50.8)
 		(end 130.6 50.8)
@@
 	)
 	(segment
-		(start 130.3 39.4)
-		(end 130.95 38.75)
+		(start 130.95 38.850001)
+		(end 130.95 37.95)
+		(width 0.2)
+		(layer "B.Cu")
+		(net 1)
+	)
+	(segment
+		(start 130.300001 39.5)
+		(end 130.95 38.850001)
 		(width 0.2)
 		(layer "B.Cu")
@@
 	)
 	(segment
-		(start 129.2 46.65)
-		(end 129.2 40.75)
+		(start 127.8 39.35)
+		(end 127.8 38.3)
 		(width 0.2)
 		(layer "B.Cu")
@@
 	)
 	(segment
-		(start 127.8 39.35)
-		(end 127.8 38.3)
+		(start 129.2 41)
+		(end 129.2 40.75)
 		(width 0.2)
 		(layer "B.Cu")
@@
 	)
 	(segment
-		(start 128.35 40.050001)
-		(end 128.350001 40.05)
-		(width 0.2)
-		(layer "F.Cu")
-		(net 4)
-	)
-	(segment
 		(start 129.8 45.5)
 		(end 129.8 47.65)
@@
 	)
 	(segment
-		(start 128.35 40.7)
-		(end 128.35 40.050001)
+		(start 128.300001 40.1)
+		(end 128.350001 40.05)
 		(width 0.2)
 		(layer "F.Cu")
@@
 	)
 	(segment
+		(start 127.8 40.1)
+		(end 128.300001 40.1)
+		(width 0.2)
+		(layer "F.Cu")
+		(net 4)
+	)
+	(segment
 		(start 131.775 47.1)
 		(end 131.4 47.1)
@@
 	)
 	(via
-		(at 128.35 40.7)
+		(at 127.8 40.1)
 		(size 0.45)
 		(drill 0.25)
@@
 	)
 	(segment
-		(start 129.8 41.6)
-		(end 128.9 40.7)
+		(start 128.75 40.1)
+		(end 129.8 41.15)
 		(width 0.2)
 		(layer "In1.Cu")
@@
 	)
 	(segment
-		(start 130.35 44.5)
-		(end 129.8 43.95)
+		(start 129.8 43.95)
+		(end 130.35 44.5)
 		(width 0.2)
 		(layer "In1.Cu")
@@
 	)
 	(segment
-		(start 129.8 43.95)
-		(end 129.8 41.6)
+		(start 129.8 41.15)
+		(end 129.8 43.95)
 		(width 0.2)
 		(layer "In1.Cu")
@@
 	)
 	(segment
-		(start 128.9 40.7)
-		(end 128.35 40.7)
+		(start 127.8 40.1)
+		(end 128.75 40.1)
 		(width 0.2)
 		(layer "In1.Cu")
