File: hardware/nfc_sense_attiny/nfc_sense.kicad_pcb (KiCad board)
At the start: 4 copper layers, 18.6 x 43.1 mm, 25 parts, among them U1 TMP117AIDRVR, U2 RF430CL330HIRGTR‎, U3 ATtiny1626-MFR

Commit message: add surface temperature version
Changed lines of the file:
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@@
 		(tags "QFN DFN_QFN")
 		(property "Reference" "U2"
-			(at 0 -2.8 90)
+			(at 2.41179 0.35 180)
 			(layer "F.SilkS")
 			(effects
