File: hardware/tools/debug/sense_debug.kicad_sch (KiCad schematic)
At the start: 53 parts, among them J1 Conn_01x03_Pin, J2 Conn_01x20_Pin, J3 Conn_01x03_Pin, J4 Conn_01x15_Pin, J5 Conn_01x12_Pin, Q1 Si1308EDL, U1 TMP117AIDRVR, U2 NTAG link, U3 ATtiny1626-MFR

Commit message: preliminary placement for debug board
Parts:
- removed C22: SUPER/HYBRIDCAP, Capacitor_SMD:C_0603_1608Metric, symbol Device:C
- added J6: B2B-PH-SM4-TB_LF__SN_, unsurv_offline_pcb_footprints:solar_2conn_solder, symbol dk_Rectangular-Connectors-Headers-Male-Pins:B2B-PH-SM4-TB_LF__SN_
- R1, R2, R4, R5: footprint Resistor_SMD:R_0402_1005Metric -> Resistor_SMD:R_0603_1608Metric
Connections:
- net ANT1: now also U2.15 (LA); no longer U2.14 (LB)
- net ANT2: now also U2.14 (LB); no longer U2.15 (LA)
- net GND: now also J6.1
- net VBAT: now also J6.2
Changed lines of the file:
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@@
 	(wire
 		(pts
-			(xy 193.04 83.82) (xy 193.04 86.36)
+			(xy 193.04 78.74) (xy 193.04 86.36)
 		)
 		(stroke
@@
 	(global_label "ANT2"
 		(shape input)
-		(at 67.31 27.94 90)
+		(at 69.85 27.94 90)
 		(fields_autoplaced yes)
 		(effects
@@
 		)
 		(property "Intersheetrefs" "${INTERSHEET_REFS}"
-			(at 67.31 20.3586 90)
+			(at 69.85 20.3586 90)
 			(effects
 				(font
@@
 	(global_label "ANT1"
 		(shape input)
-		(at 69.85 27.94 90)
+		(at 67.31 27.94 90)
 		(fields_autoplaced yes)
 		(effects
@@
 		)
 		(property "Intersheetrefs" "${INTERSHEET_REFS}"
-			(at 69.9294 20.9307 90)
+			(at 67.3894 20.9307 90)
 			(effects
 				(font
@@
 	)
 	(symbol
-		(lib_id "Connector:TestPoint")
-		(at 250.19 76.2 0)
+		(lib_id "dk_Rectangular-Connectors-Headers-Male-Pins:B2B-PH-SM4-TB_LF__SN_")
+		(at 195.58 78.74 90)
 		(unit 1)
 		(exclude_from_sim no)
@@
 		(dnp no)
 		(fields_autoplaced yes)
-		(property "Reference" "TP3"
-			(at 251.587 72.0633 0)
+		(property "Reference" "J6"
+			(at 198.755 76.2578 90)
 			(effects
 				(font
 					(size 1.27 1.27)
 				)
-				(justify left)
+				(justify right)
 			)
 		)
-		(property "Value" "TestPoint"
-			(at 251.587 74.6002 0)
+		(property "Value" "B2B-PH-SM4-TB_LF__SN_"
+			(at 198.755 78.6821 90)
 			(effects
 				(font
 					(size 1.27 1.27)
 				)
+				(justify right)
+			)
+		)
+		(property "Footprint" "unsurv_offline_pcb_footprints:solar_2conn_solder"
+			(at 190.5 73.66 0)
+			(effects
+				(font
+					(size 1.524 1.524)
+				)
 				(justify left)
+				(hide yes)
 			)
 		)
-		(property "Footprint" "TestPoint:TestPoint_Pad_D1.0mm"
-			(at 255.27 76.2 0)
+		(property "Datasheet" "http://www.jst-mfg.com/product/pdf/eng/ePH.pdf"
+			(at 187.96 73.66 0)
 			(effects
 				(font
-					(size 1.27 1.27)
+					(size 1.524 1.524)
 				)
+				(justify left)
 				(hide yes)
 			)
 		)
-		(property "Datasheet" "~"
-			(at 255.27 76.2 0)
+		(property "Description" "CONN HEADER SMD 2POS 2MM"
+			(at 195.58 78.74 0)
 			(effects
 				(font
@@
 			)
 		)
-		(property "Description" ""
-			(at 250.19 76.2 0)
+		(property "Digi-Key_PN" "455-1734-1-ND"
+			(at 185.42 73.66 0)
 			(effects
 				(font
-					(size 1.27 1.27)
+					(size 1.524 1.524)
+				)
+				(justify left)
+				(hide yes)
+			)
+		)
+		(property "MPN" "B2B-PH-SM4-TB(LF)(SN)"
+			(at 182.88 73.66 0)
+			(effects
+				(font
+					(size 1.524 1.524)
+				)
+				(justify left)
+				(hide yes)
+			)
+		)
+		(property "Category" "Connectors, Interconnects"
+			(at 180.34 73.66 0)
+			(effects
+				(font
+					(size 1.524 1.524)
+				)
+				(justify left)
+				(hide yes)
+			)
+		)
+		(property "Family" "Rectangular Connectors - Headers, Male Pins"
+			(at 177.8 73.66 0)
+			(effects
+				(font
+					(size 1.524 1.524)
+				)
+				(justify left)
+				(hide yes)
+			)
+		)
+		(property "DK_Datasheet_Link" "http://www.jst-mfg.com/product/pdf/eng/ePH.pdf"
+			(at 175.26 73.66 0)
+			(effects
+				(font
+					(size 1.524 1.524)
+				)
+				(justify left)
+				(hide yes)
+			)
+		)
+		(property "DK_Detail_Page" "/product-detail/en/jst-sales-america-inc/B2B-PH-SM4-TB(LF)(SN)/455-1734-1-ND/926831"
+			(at 172.72 73.66 0)
+			(effects
+				(font
+					(size 1.524 1.524)
+				)
+				(justify left)
+				(hide yes)
+			)
+		)
+		(property "Description_1" "CONN HEADER SMD 2POS 2MM"
+			(at 170.18 73.66 0)
+			(effects
+				(font
+					(size 1.524 1.524)
+				)
+				(justify left)
+				(hide yes)
+			)
+		)
+		(property "Manufacturer" "JST Sales America Inc."
+			(at 167.64 73.66 0)
+			(effects
+				(font
+					(size 1.524 1.524)
+				)
+				(justify left)
+				(hide yes)
+			)
+		)
+		(property "Status" "Active"
+			(at 165.1 73.66 0)
+			(effects
+				(font
+					(size 1.524 1.524)
 				)
+				(justify left)
 				(hide yes)
 			)
@@
 		(pin "1"
 		)
+		(pin "2"
+		)
 		(instances
-			(project "pocket_knife_sense_display"
+			(project ""
 				(path "/c54e1377-ff88-4224-9c85-352a20bf3450"
-					(reference "TP3")
+					(reference "J6")
 					(unit 1)
 				)
@@
 	)
 	(symbol
-		(lib_id "power:GND")
-		(at 223.52 153.67 0)
+		(lib_id "Connector:TestPoint")
+		(at 250.19 76.2 0)
 		(unit 1)
 		(exclude_from_sim no)
@@
 		(dnp no)
 		(fields_autoplaced yes)
-		(property "Reference" "#PWR015"
-			(at 223.52 160.02 0)
+		(property "Reference" "TP3"
+			(at 251.587 72.0633 0)
 			(effects
 				(font
 					(size 1.27 1.27)
 				)
-				(hide yes)
+				(justify left)
 			)
 		)
-		(property "Value" "GND"
-			(at 223.52 158.1134 0)
+		(property "Value" "TestPoint"
+			(at 251.587 74.6002 0)
 			(effects
 				(font
 					(size 1.27 1.27)
 				)
+				(justify left)
 			)
 		)
-		(property "Footprint" ""
-			(at 223.52 153.67 0)
+		(property "Footprint" "TestPoint:TestPoint_Pad_D1.0mm"
+			(at 255.27 76.2 0)
 			(effects
 				(font
@@
 			)
 		)
-		(property "Datasheet" ""
-			(at 223.52 153.67 0)
+		(property "Datasheet" "~"
+			(at 255.27 76.2 0)
 			(effects
 				(font
@@
 		)
 		(property "Description" ""
-			(at 223.52 153.67 0)
+			(at 250.19 76.2 0)
 			(effects
 				(font
@@
 			(project "pocket_knife_sense_display"
 				(path "/c54e1377-ff88-4224-9c85-352a20bf3450"
-					(reference "#PWR015")
+					(reference "TP3")
 					(unit 1)
 				)
@@
 	)
 	(symbol
-		(lib_id "Device:C_Small")
-		(at 172.72 90.17 90)
+		(lib_id "power:GND")
+		(at 223.52 153.67 0)
 		(unit 1)
 		(exclude_from_sim no)
@@
 		(dnp no)
 		(fields_autoplaced yes)
-		(property "Reference" "C21"
-			(at 172.7263 84.4634 90)
+		(property "Reference" "#PWR015"
+			(at 223.52 160.02 0)
 			(effects
 				(font
 					(size 1.27 1.27)
 				)
+				(hide yes)
 			)
 		)
-		(property "Value" "47uF"
-			(at 172.7263 86.8877 90)
+		(property "Value" "GND"
+			(at 223.52 158.1134 0)
 			(effects
 				(font
@@
 			)
 		)
-		(property "Footprint" "Capacitor_SMD:C_0603_1608Metric"
-			(at 172.72 90.17 0)
+		(property "Footprint" ""
+			(at 223.52 153.67 0)
 			(effects
 				(font
@@
 			)
 		)
-		(property "Datasheet" "~"
-			(at 172.72 90.17 0)
+		(property "Datasheet" ""
+			(at 223.52 153.67 0)
 			(effects
 				(font
@@
 			)
 		)
-		(property "Description" "Unpolarized capacitor, small symbol"
-			(at 172.72 90.17 0)
+		(property "Description" ""
+			(at 223.52 153.67 0)
 			(effects
 				(font
@@
 		(pin "1"
 		)
-		(pin "2"
-		)
 		(instances
-			(project "sense_debug"
+			(project "pocket_knife_sense_display"
 				(path "/c54e1377-ff88-4224-9c85-352a20bf3450"
-					(reference "C21")
+					(reference "#PWR015")
 					(unit 1)
 				)
@@
 	)
 	(symbol
-		(lib_id "Device:C")
-		(at 193.04 80.01 0)
+		(lib_id "Device:C_Small")
+		(at 172.72 90.17 90)
 		(unit 1)
 		(exclude_from_sim no)
@@
 		(dnp no)
 		(fields_autoplaced yes)
-		(property "Reference" "C22"
-			(at 195.961 78.7978 0)
+		(property "Reference" "C21"
+			(at 172.7263 84.4634 90)
 			(effects
 				(font
 					(size 1.27 1.27)
 				)
-				(justify left)
 			)
 		)
-		(property "Value" "SUPER/HYBRIDCAP"
-			(at 195.961 81.2221 0)
+		(property "Value" "47uF"
+			(at 172.7263 86.8877 90)
 			(effects
 				(font
 					(size 1.27 1.27)
 				)
-				(justify left)
 			)
 		)
 		(property "Footprint" "Capacitor_SMD:C_0603_1608Metric"
-			(at 194.0052 83.82 0)
+			(at 172.72 90.17 0)
 			(effects
 				(font
@@
 		)
 		(property "Datasheet" "~"
-			(at 193.04 80.01 0)
+			(at 172.72 90.17 0)
 			(effects
 				(font
@@
 			)
 		)
-		(property "Description" "Unpolarized capacitor"
-			(at 193.04 80.01 0)
+		(property "Description" "Unpolarized capacitor, small symbol"
+			(at 172.72 90.17 0)
 			(effects
 				(font
@@
 			)
 		)
-		(pin "2"
-		)
 		(pin "1"
 		)
+		(pin "2"
+		)
 		(instances
-			(project ""
+			(project "sense_debug"
 				(path "/c54e1377-ff88-4224-9c85-352a20bf3450"
-					(reference "C22")
+					(reference "C21")
 					(unit 1)
 				)
@@
 			)
 		)
-		(property "Footprint" "Resistor_SMD:R_0402_1005Metric"
+		(property "Footprint" "Resistor_SMD:R_0603_1608Metric"
 			(at 26.162 153.67 90)
 			(effects
@@
 			)
 		)
-		(property "Footprint" "Resistor_SMD:R_0402_1005Metric"
+		(property "Footprint" "Resistor_SMD:R_0603_1608Metric"
 			(at 186.182 153.67 90)
 			(effects
@@
 			)
 		)
-		(property "Footprint" "Resistor_SMD:R_0402_1005Metric"
+		(property "Footprint" "Resistor_SMD:R_0603_1608Metric"
 			(at 16.002 153.67 90)
 			(effects
@@
 			)
 		)
-		(property "Footprint" "Resistor_SMD:R_0402_1005Metric"
+		(property "Footprint" "Resistor_SMD:R_0603_1608Metric"
 			(at 178.562 153.67 90)
 			(effects

Commit message: route debug board
Parts:
- added J7: Conn_01x03_Pin, Connector_PinHeader_2.54mm:PinHeader_1x03_P2.54mm_Vertical, symbol Connector:Conn_01x03_Pin
Connections:
- net GND: now also J7.3 (Pin_3)
- net PREVGH: now also D2.2 (A); no longer D2.1 (K)
- net RX: now also J7.1 (Pin_1)
- net TX: now also J7.2 (Pin_2)
- net VIN: no longer J5.3 (Pin_3)
- net VLDO: no longer J5.2 (Pin_2)
- net at C11.1, L1.2, Q1.3 (D): now also D2.1 (K); no longer D2.2 (A)
Other:
- note added: "TODO - connect SPI for display - power harvesting conn - PH super / hybrid cap - power rail jumpers - particle sensor conn - external debug conn - SERIAL CONN OUT!!!"
- note removed: "TODO - connect SPI for display - power harvesting conn - PH super / hybrid cap - power rail jumpers - particle sensor conn - external debug conn"
- moved on the sheet: D2, J6
