File: hardware/tools/debug/sense_debug.kicad_sch (KiCad schematic)
At the start: 54 parts, among them J1 Conn_01x03_Pin, J2 Conn_01x20_Pin, J3 Conn_01x03_Pin, J4 Conn_01x15_Pin, J5 Conn_01x12_Pin, J6 B2B-PH-SM4-TB_LF__SN_, J7 Conn_01x03_Pin, Q1 Si1308EDL, U1 TMP117AIDRVR, U2 NTAG link, U3 ATtiny1626-MFR

Commit message: update nfc sense ntag with attiny 1626
Parts:
- U4: value ~ -> (none)
